File: hardware/RC-Multiswitch-ESP32-S3.kicad_sch (KiCad schematic)
At the start: 32 parts, among them CN1 UART A, CN2 5-12V, J1 Ausgaenge, J5 UART B, J6 UART C, U1 ESP32-S3-Zero, U2 ULN2803A

Commit message: Hardware: NEG- und POS-Variante (TBD62783APG), UART-Beschriftung korrigiert
- Neues KiCad-Projekt RC-Multiswitch-ESP32-S3-NEG: ULN2803A, Platine 1:1 wie Original
- Neues KiCad-Projekt RC-Multiswitch-ESP32-S3-POS: positiv schaltend mit TBD62783APG
  (U2 Pin 9 = VLOAD, Pin 10 = GND, J1-Schiene auf GND, drei Bahnen an U2, Bestueckungsdruck)
- Original-Schaltplan v0.4: UART B/C RX/TX-Labels passend zu Platine und Firmware
- README-hardware: Abschnitt zu den Varianten

Co-Authored-By: Claude Opus 5.5 <noreply@anthropic.com>
Claude-Session: https://claude.ai/code/session_0118D4qppRkb6gR5m3R2CZyV
Connections:
- net UB_RX: now also U1.13 (IO12); no longer U1.12 (IO13)
- net UB_TX: now also U1.12 (IO13); no longer U1.13 (IO12)
- net UC_RX: now also U1.4 (IO1); no longer U1.5 (IO2)
- net UC_TX: now also U1.5 (IO2); no longer U1.4 (IO1)
Changed lines of the file:
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@@
 		(title "RC Multiswitch ESP32-S3-Zero (ULN2803A)")
 		(date "2026-10-14")
-		(rev "v0.3")
+		(rev "v0.4")
 		(comment 1 "Entwurf - vor Layout/Bestellung pruefen")
 	)
@@
 		)
 	)
-	(label "UB_RX"
+	(label "UB_TX"
 		(at 93.98 111.76 0)
 		(effects
@@
 		)
 	)
-	(label "UB_TX"
+	(label "UB_RX"
 		(at 93.98 114.3 0)
 		(effects
@@
 		)
 	)
-	(label "UC_TX"
+	(label "UC_RX"
 		(at 93.98 121.92 0)
 		(effects
@@
 		)
 	)
-	(label "UC_RX"
+	(label "UC_TX"
 		(at 93.98 119.38 0)
 		(effects
