File: hardware/RC-Multiswitch-ESP32-S3-NEG.kicad_pcb (KiCad board)
At the start: 2 copper layers, 66.5 x 50.6 mm, 33 parts, among them CN1 UART A, CN2 5-12V, J1 Ausgaenge, J5 J5_UART B, J6 UART C, U1 ESP32-S3-Zero, U2 ULN2803A

Commit message: Hardware: TBD62083APG statt ULN2803A, Original-Projekt entfernt
ULN2803A ist abgekuendigt. Der TBD62083APG (DMOS) hat dieselbe Pinbelegung und passt in denselben Sockel, Leiterbahnen und Netze bleiben unveraendert. Schaltplan-Symbol, Bauteilwert, Bestueckungsdruck und Doku angepasst.

Co-Authored-By: Claude Opus 5.5 <noreply@anthropic.com>
Claude-Session: https://claude.ai/code/session_0118D4qppRkb6gR5m3R2CZyV
Parts:
- U2: value ULN2803A -> TBD62083APG
Other:
- board text added: "TBD62083APG"
- board text removed: "ULN2803A"
Changed lines of the file:
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@@
 			)
 		)
-		(property "Value" "ULN2803A"
+		(property "Value" "TBD62083APG"
 			(at 3.81 23.67 0)
 			(layer "F.Fab")
@@
 		)
 	)
-	(gr_text "ULN2803A"
+	(gr_text "TBD62083APG"
 		(at 156.5 85.5 0)
 		(layer "F.SilkS")
