File: hardware/RC-Multiswitch-ESP32-S3-POS.kicad_sch (KiCad schematic)
At the start: 32 parts, among them CN1 UART A, CN2 5-12V, J1 Ausgaenge, J5 UART B, J6 UART C, U1 ESP32-S3-Zero, U2 TBD62783APG

Commit message: Hardware: TBD62083APG statt ULN2803A, Original-Projekt entfernt
ULN2803A ist abgekuendigt. Der TBD62083APG (DMOS) hat dieselbe Pinbelegung und passt in denselben Sockel, Leiterbahnen und Netze bleiben unveraendert. Schaltplan-Symbol, Bauteilwert, Bestueckungsdruck und Doku angepasst.

Co-Authored-By: Claude Opus 5.5 <noreply@anthropic.com>
Claude-Session: https://claude.ai/code/session_0118D4qppRkb6gR5m3R2CZyV
Other:
- note added: "Last: 5-12V, Verbraucher zwischen OUTn und GND. Max. 500mA je Kanal, Summe aller Kanaele max. ca. 1,5A. NICHT mit ULN2803A/TBD62083APG bestuecken (Pin 9/10 anders). ESP32 wird aus +5V von CN1 (BEC/Empfaenger) versorgt. Adresse per Firmware/Web-UI/Lua. Keine Pulldowns, keine UART-Vorwiderstaende. R1-R16: Werte legt der Anwender je LED bzw. Verbraucher selbst aus (siehe Projektbeschreibung)."
- note removed: "Last: 5-12V, Verbraucher zwischen OUTn und GND. Max. 500mA je Kanal, Summe aller Kanaele max. ca. 1,5A. NICHT mit ULN2803 bestuecken (Pin 9/10 anders). ESP32 wird aus +5V von CN1 (BEC/Empfaenger) versorgt. Adresse per Firmware/Web-UI/Lua. Keine Pulldowns, keine UART-Vorwiderstaende. R1-R16: Werte legt der Anwender je LED bzw. Verbraucher selbst aus (siehe Projektbeschreibung)."
Changed lines of the file:
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@@
 		)
 	)
-	(text "Last: 5-12V, Verbraucher zwischen OUTn und GND. Max. 500mA je Kanal, Summe aller Kanaele max. ca. 1,5A. NICHT mit ULN2803 bestuecken (Pin 9/10 anders). ESP32 wird aus +5V von CN1 (BEC/Empfaenger) versorgt. Adresse per Firmware/Web-UI/Lua. Keine Pulldowns, keine UART-Vorwiderstaende. R1-R16: Werte legt der Anwender je LED bzw. Verbraucher selbst aus (siehe Projektbeschreibung)."
+	(text "Last: 5-12V, Verbraucher zwischen OUTn und GND. Max. 500mA je Kanal, Summe aller Kanaele max. ca. 1,5A. NICHT mit ULN2803A/TBD62083APG bestuecken (Pin 9/10 anders). ESP32 wird aus +5V von CN1 (BEC/Empfaenger) versorgt. Adresse per Firmware/Web-UI/Lua. Keine Pulldowns, keine UART-Vorwiderstaende. R1-R16: Werte legt der Anwender je LED bzw. Verbraucher selbst aus (siehe Projektbeschreibung)."
 		(exclude_from_sim no)
 		(at 15 21 0)
